File: MCU.sch (KiCad schematic (older format))
At the start: 23 parts, among them J2 JTAG, J3 BOOT, U6 STM32F303RETx

Commit message: Fixed most ERC errors
Connections:
- net labels removed: ACT, ADC, I2C1, SPI1, SPI2, SWDIO-JTCK, SWDIO-JTMS, USART1_2
- no-connect marks 0 -> 22
Changed lines of the file:
@@
 $Descr USLetter 11000 8500
 encoding utf-8
-Sheet 2 3
+Sheet 3 3
 Title "Flight Computer"
 Date ""
@@
 	4000 2250 4000 2450
 Connection ~ 4000 2450
-Text Label 6450 2950 0    60   ~ 0
-SPI1_SCK
-Text Label 6450 3050 0    60   ~ 0
-SPI1_MISO
-Text Label 6450 3150 0    60   ~ 0
-SPI1_MOSI
-Entry Wire Line
-	7000 2950 7100 3050
-Entry Wire Line
-	7000 3050 7100 3150
-Entry Wire Line
-	7000 3150 7100 3250
 Wire Wire Line
 	6400 2950 7000 2950
@@
 Wire Wire Line
 	6400 3150 7000 3150
-Text Label 6450 2450 0    60   ~ 0
-ADC1
-Text Label 6450 2550 0    60   ~ 0
-ADC2
-Text Label 6450 2650 0    60   ~ 0
-ADC3
-Text Label 6450 2750 0    60   ~ 0
-ADC4
 Wire Wire Line
 	6400 4450 6450 4450
@@
 Wire Wire Line
 	6400 4850 7000 4850
-Text Label 6450 4450 0    60   ~ 0
-USART2_TX
-Text Label 6450 4550 0    60   ~ 0
-USART2_RX
-Text Label 6450 4750 0    60   ~ 0
-USART1_TX
-Text Label 6450 4850 0    60   ~ 0
-USART1_RX
-Entry Wire Line
-	7000 4450 7100 4550
-Entry Wire Line
-	7000 4550 7100 4650
-Entry Wire Line
-	7000 4750 7100 4850
-Entry Wire Line
-	7000 4850 7100 4950
 Wire Wire Line
 	6400 3250 7000 3250
@@
 Wire Wire Line
 	6400 3550 7000 3550
-Text Label 6450 3250 0    60   ~ 0
-SPI1_CS1
-Text Label 6450 3350 0    60   ~ 0
-SPI1_CS2
-Text Label 6450 3450 0    60   ~ 0
-SPI1_CS3
-Text Label 6450 3550 0    60   ~ 0
-SPI1_CS4
-Entry Wire Line
-	7000 3250 7100 3350
-Entry Wire Line
-	7000 3350 7100 3450
-Entry Wire Line
-	7000 3450 7100 3550
-Entry Wire Line
-	7000 3550 7100 3650
 $Comp
 L Diode:BAT54S D3
@@
 L power:GND #PWR032
 U 1 1 5E211E73
-P 8800 2400
-F 0 "#PWR032" H 8800 2150 50  0001 C CNN
-F 1 "GND" H 8800 2250 50  0000 C CNN
-F 2 "" H 8800 2400 50  0001 C CNN
-F 3 "" H 8800 2400 50  0001 C CNN
-	1    8800 2400
+P 8800 2250
+F 0 "#PWR032" H 8800 2000 50  0001 C CNN
+F 1 "GND" H 8800 2100 50  0000 C CNN
+F 2 "" H 8800 2250 50  0001 C CNN
+F 3 "" H 8800 2250 50  0001 C CNN
+	1    8800 2250
 	1    0    0    -1
 $EndComp
@@
 	6400 2450 7200 2450
 Connection ~ 7200 2400
-Wire Wire Line
-	7600 2100 7600 2550
-Wire Wire Line
-	6400 2550 7600 2550
 Connection ~ 7600 2100
 Wire Wire Line
@@
 	7500 2200 8800 2200
 Wire Wire Line
-	8800 2200 8800 2400
+	8800 2200 8800 2250
 Connection ~ 7500 2200
 Wire Wire Line
@@
 Wire Wire Line
 	6400 5350 7000 5350
-Entry Wire Line
-	7000 5350 7100 5450
-Entry Wire Line
-	7000 5450 7100 5550
-Entry Wire Line
-	7000 5550 7100 5650
-Entry Wire Line
-	7000 5650 7100 5750
-Text Label 6450 5650 0    60   ~ 0
-SPI2_MOSI
-Text Label 6450 5550 0    60   ~ 0
-SPI2_MISO
-Text Label 6450 5450 0    60   ~ 0
-SPI2_SCK
-Text Label 6450 5350 0    60   ~ 0
-SPI2_CS2
 Wire Wire Line
 	6400 5250 7000 5250
-Text Label 6450 5250 0    60   ~ 0
-SPI2_CS1
-Entry Wire Line
-	7000 5250 7100 5350
-Wire Bus Line
-	7100 3700 9100 3700
-Wire Bus Line
-	7100 5000 9100 5000
 Wire Wire Line
 	6400 4950 7000 4950
 Wire Wire Line
 	6400 5050 7000 5050
-Text Label 6450 4950 0    60   ~ 0
-I2C1_SDA
-Text Label 6450 5050 0    60   ~ 0
-I2C1_SCL
-Text HLabel 9100 5000 2    60   BiDi ~ 12
-USART1_2
-Text HLabel 9100 3700 2    60   BiDi ~ 12
-SPI1
-Wire Bus Line
-	7100 5200 9100 5200
-Entry Wire Line
-	7000 4950 7100 5050
-Entry Wire Line
-	7000 5050 7100 5150
-Text HLabel 9100 5200 2    60   BiDi ~ 12
-I2C1
-Entry Wire Line
-	8000 2900 8100 3000
-Entry Wire Line
-	7600 2900 7700 3000
-Entry Wire Line
-	7200 2900 7300 3000
-Entry Wire Line
-	8400 2900 8500 3000
-Wire Wire Line
-	7200 2450 7200 2900
-Connection ~ 7200 2450
-Wire Wire Line
-	7600 2550 7600 2900
-Connection ~ 7600 2550
-Wire Wire Line
-	8000 2650 8000 2900
-Connection ~ 8000 2650
-Wire Wire Line
-	8400 2750 8400 2900
-Connection ~ 8400 2750
-Text HLabel 9100 3000 2    60   BiDi ~ 12
-ADC
 Wire Wire Line
 	1950 1700 1350 1700
@@
 Wire Wire Line
 	5000 4450 4400 4450
-Text Label 4500 4150 0    60   ~ 0
-ACT1
-Text Label 4500 4250 0    60   ~ 0
-ACT2
-Text Label 4500 4350 0    60   ~ 0
-ACT3
-Text Label 4500 4450 0    60   ~ 0
-ACT4
-Entry Wire Line
-	4400 4150 4300 4250
-Entry Wire Line
-	4400 4250 4300 4350
-Entry Wire Line
-	4400 4350 4300 4450
-Entry Wire Line
-	4400 4450 4300 4550
-Wire Bus Line
-	4300 4600 3500 4600
-Text HLabel 3500 4600 0    60   BiDi ~ 12
-ACT
-Text HLabel 9100 5800 2    60   BiDi ~ 12
-SPI2
-Wire Bus Line
-	7100 5800 9100 5800
 $Comp
 L Connector_Generic:Conn_01x03 J3
@@
 	6400 3750 7000 3750
 Text Label 6450 3750 0    60   ~ 0
-SWDIO-JTMS
+SWDIO_JTMS
 Text Label 6450 3850 0    60   ~ 0
-SWDIO-JTCK
+SWDIO_JTCK
 Text Label 6450 3950 0    60   ~ 0
 JTDI
@@
 Wire Wire Line
 	2550 1700 2550 1950
-Wire Bus Line
-	7100 5050 7100 5200
-Wire Bus Line
-	4300 4250 4300 4600
-Wire Bus Line
-	7300 3000 9100 3000
-Wire Bus Line
-	7100 5350 7100 5800
-Wire Bus Line
-	7100 4550 7100 5000
-Wire Bus Line
-	7100 3050 7100 3700
+NoConn ~ 6400 4150
+NoConn ~ 6400 4250
+NoConn ~ 6400 3650
+NoConn ~ 5000 3650
+NoConn ~ 5000 3750
+NoConn ~ 5000 3950
+NoConn ~ 5000 4550
+NoConn ~ 5000 4650
+NoConn ~ 5000 4750
+NoConn ~ 5000 4850
+NoConn ~ 5000 4950
+NoConn ~ 5000 5050
+NoConn ~ 5000 5150
+NoConn ~ 5000 5250
+NoConn ~ 5000 5350
+NoConn ~ 6400 5150
+NoConn ~ 6400 4650
+NoConn ~ 6400 4350
+NoConn ~ 5000 5450
+NoConn ~ 5000 5550
+NoConn ~ 5000 5650
+Text HLabel 4400 4150 0    60   BiDi ~ 0
+ACT1
+Text HLabel 4400 4250 0    60   BiDi ~ 0
+ACT2
+Text HLabel 4400 4350 0    60   BiDi ~ 0
+ACT3
+Text HLabel 4400 4450 0    60   BiDi ~ 0
+ACT4
+Text HLabel 7000 4450 2    60   BiDi ~ 0
+USART2_TX
+Text HLabel 7000 4550 2    60   BiDi ~ 0
+USART2_RX
+Text HLabel 7000 4750 2    60   BiDi ~ 0
+USART1_TX
+Text HLabel 7000 4850 2    60   BiDi ~ 0
+USART1_RX
+Text HLabel 7000 4950 2    60   BiDi ~ 0
+I2C1_SDA
+Text HLabel 7000 5050 2    60   BiDi ~ 0
+I2C1_SCL
+Text HLabel 7000 5250 2    60   BiDi ~ 0
+SPI2_CS1
+Text HLabel 7000 5350 2    60   BiDi ~ 0
+SPI2_CS2
+Text HLabel 7000 5450 2    60   BiDi ~ 0
+SPI2_SCK
+Text HLabel 7000 5550 2    60   BiDi ~ 0
+SPI2_MISO
+Text HLabel 7000 5650 2    60   BiDi ~ 0
+SPI2_MOSI
+Wire Wire Line
+	7600 2100 7600 2550
+Wire Wire Line
+	7200 2450 9000 2450
+Connection ~ 7200 2450
+Wire Wire Line
+	7600 2550 9000 2550
+Wire Wire Line
+	8000 2650 9000 2650
+Connection ~ 8000 2650
+Wire Wire Line
+	8400 2750 9000 2750
+Connection ~ 8400 2750
+Connection ~ 7600 2550
+Wire Wire Line
+	6400 2550 7600 2550
+NoConn ~ 6400 2850
+Text HLabel 7000 2950 2    60   BiDi ~ 0
+SPI1_SCK
+Text HLabel 7000 3050 2    60   BiDi ~ 0
+SPI1_MISO
+Text HLabel 7000 3150 2    60   BiDi ~ 0
+SPI1_MOSI
+Text HLabel 7000 3250 2    60   BiDi ~ 0
+SPI1_CS1
+Text HLabel 7000 3350 2    60   BiDi ~ 0
+SPI1_CS2
+Text HLabel 7000 3450 2    60   BiDi ~ 0
+SPI1_CS3
+Text HLabel 7000 3550 2    60   BiDi ~ 0
+SPI1_CS4
+Text HLabel 9000 2450 2    60   BiDi ~ 0
+ADC1
+Text HLabel 9000 2550 2    60   BiDi ~ 0
+ADC2
+Text HLabel 9000 2650 2    60   BiDi ~ 0
+ADC3
+Text HLabel 9000 2750 2    60   BiDi ~ 0
+ADC4
 $EndSCHEMATC

Commit message: Removed redundant ADC protection diodes Basic PCB component layout
Parts:
- removed G2: LOGO, Flight-Computer:UB-SEDS-Logo, symbol Flight-Computer:UB-SEDS-Logo
Changed lines of the file:
@@
 $EndDescr
-$Comp
-L Flight-Computer:UB-SEDS-Logo G2
-U 1 1 5CB119A1
-P 9850 7100
-F 0 "G2" H 9850 6963 60  0001 C CNN
-F 1 "LOGO" H 9850 7237 60  0001 C CNN
-F 2 "Flight-Computer:UB-SEDS-Logo" H 9850 7100 60  0001 C CNN
-F 3 "" H 9850 7100 60  0001 C CNN
-	1    9850 7100
-	1    0    0    -1
-$EndComp
 $Comp
 L MCU_ST_STM32F3:STM32F303RETx U6

Commit message: Renamed some components?
Parts:
- removed D2, D4, D6, D8: BAT54S, Package_TO_SOT_SMD:SOT-23, symbol Diode:BAT54S
- renumbered D3 to D2, D5 to D3, D7 to D4, R5 to R12, R6 to R13, R7 to R14, R8 to R15
Changed lines of the file:
@@
 $EndComp
 $Comp
-L power:+3V3 #PWR030
+L power:+3V3 #PWR035
 U 1 1 5DF125E2
 P 6000 1550
-F 0 "#PWR030" H 6000 1400 50  0001 C CNN
+F 0 "#PWR035" H 6000 1400 50  0001 C CNN
 F 1 "+3V3" H 6000 1690 50  0000 C CNN
 F 2 "" H 6000 1550 50  0001 C CNN
@@
 $EndComp
 $Comp
-L power:GND #PWR029
+L power:GND #PWR034
 U 1 1 5DF17C0F
 P 5900 6350
-F 0 "#PWR029" H 5900 6100 50  0001 C CNN
+F 0 "#PWR034" H 5900 6100 50  0001 C CNN
 F 1 "GND" H 5900 6200 50  0000 C CNN
 F 2 "" H 5900 6350 50  0001 C CNN
@@
 	5500 1700 5500 2250
 $Comp
-L power:GND #PWR028
+L power:GND #PWR033
 U 1 1 5DFA0210
 P 4000 3150
-F 0 "#PWR028" H 4000 2900 50  0001 C CNN
+F 0 "#PWR033" H 4000 2900 50  0001 C CNN
 F 1 "GND" H 4000 3000 50  0000 C CNN
 F 2 "" H 4000 3150 50  0001 C CNN
@@
 	6400 3550 7000 3550
 $Comp
-L Diode:BAT54S D3
+L Diode:BAT54S D2
 U 1 1 5E142556
 P 7600 1900
-F 0 "D3" V 7554 1988 50  0000 L CNN
+F 0 "D2" V 7554 1988 50  0000 L CNN
 F 1 "BAT54S" V 7645 1988 50  0000 L CNN
 F 2 "Package_TO_SOT_SMD:SOT-23" H 7675 2025 50  0001 L CNN
@@
 $EndComp
 $Comp
-L Diode:BAT54S D4
-U 1 1 5E14255C
-P 7600 1900
-F 0 "D4" V 7554 1988 50  0000 L CNN
-F 1 "BAT54S" V 7645 1988 50  0000 L CNN
-F 2 "Package_TO_SOT_SMD:SOT-23" H 7675 2025 50  0001 L CNN
-F 3 "https://www.diodes.com/assets/Datasheets/ds11005.pdf" H 7480 1900 50  0001 C CNN
-	1    7600 1900
-	-1   0    0    -1
-$EndComp
-$Comp
-L Diode:BAT54S D5
-U 1 1 5E211E6E
-P 8000 1600
-F 0 "D5" V 7954 1688 50  0000 L CNN
-F 1 "BAT54S" V 8045 1688 50  0000 L CNN
-F 2 "Package_TO_SOT_SMD:SOT-23" H 8075 1725 50  0001 L CNN
-F 3 "https://www.diodes.com/assets/Datasheets/ds11005.pdf" H 7880 1600 50  0001 C CNN
-	1    8000 1600
-	-1   0    0    -1
-$EndComp
-$Comp
-L Diode:BAT54S D6
-U 1 1 5E211E6F
-P 8000 1600
-F 0 "D6" V 7954 1688 50  0000 L CNN
-F 1 "BAT54S" V 8045 1688 50  0000 L CNN
-F 2 "Package_TO_SOT_SMD:SOT-23" H 8075 1725 50  0001 L CNN
-F 3 "https://www.diodes.com/assets/Datasheets/ds11005.pdf" H 7880 1600 50  0001 C CNN
-	1    8000 1600
-	-1   0    0    -1
-$EndComp
-$Comp
-L power:+3V3 #PWR031
+L power:+3V3 #PWR036
 U 1 1 5E211E72
 P 6800 1100
-F 0 "#PWR031" H 6800 950 50  0001 C CNN
+F 0 "#PWR036" H 6800 950 50  0001 C CNN
 F 1 "+3V3" H 6800 1240 50  0000 C CNN
 F 2 "" H 6800 1100 50  0001 C CNN
@@
 $EndComp
 $Comp
-L power:GND #PWR032
+L power:GND #PWR037
 U 1 1 5E211E73
 P 8800 2250
-F 0 "#PWR032" H 8800 2000 50  0001 C CNN
+F 0 "#PWR037" H 8800 2000 50  0001 C CNN
 F 1 "GND" H 8800 2100 50  0000 C CNN
 F 2 "" H 8800 2250 50  0001 C CNN
@@
 	1    8800 2250
 	1    0    0    -1
-$EndComp
-$Comp
-L Diode:BAT54S D2
-U 1 1 5E211E6B
-P 7200 2200
-F 0 "D2" V 7154 2288 50  0000 L CNN
-F 1 "BAT54S" V 7245 2288 50  0000 L CNN
-F 2 "Package_TO_SOT_SMD:SOT-23" H 7275 2325 50  0001 L CNN
-F 3 "https://www.diodes.com/assets/Datasheets/ds11005.pdf" H 7080 2200 50  0001 C CNN
-	1    7200 2200
-	-1   0    0    -1
 $EndComp
 $Comp
@@
 	-1   0    0    -1
 $EndComp
-$Comp
-L Diode:BAT54S D7
-U 1 1 5E211E70
-P 8400 1300
-F 0 "D7" V 8354 1388 50  0000 L CNN
-F 1 "BAT54S" V 8445 1388 50  0000 L CNN
-F 2 "Package_TO_SOT_SMD:SOT-23" H 8475 1425 50  0001 L CNN
-F 3 "https://www.diodes.com/assets/Datasheets/ds11005.pdf" H 8280 1300 50  0001 C CNN
-	1    8400 1300
-	-1   0    0    -1
-$EndComp
-$Comp
-L Diode:BAT54S D8
-U 1 1 5E211E71
-P 8400 1300
-F 0 "D8" V 8354 1388 50  0000 L CNN
-F 1 "BAT54S" V 8445 1388 50  0000 L CNN
-F 2 "Package_TO_SOT_SMD:SOT-23" H 8475 1425 50  0001 L CNN
-F 3 "https://www.diodes.com/assets/Datasheets/ds11005.pdf" H 8280 1300 50  0001 C CNN
-	1    8400 1300
-	-1   0    0    -1
-$EndComp
 Wire Wire Line
 	6000 1700 6000 2100
@@
 	4000 1700 4000 1950
 $Comp
-L Device:R R8
+L Device:R R15
 U 1 1 5DFE6933
 P 4000 2100
-F 0 "R8" V 4080 2100 50  0000 C CNN
+F 0 "R15" V 4080 2100 50  0000 C CNN
 F 1 "10k" V 4000 2100 50  0000 C CNN
 F 2 "Resistor_SMD:R_1206_3216Metric_Pad1.42x1.75mm_HandSolder" V 3930 2100 50  0001 C CNN
@@
 Wire Wire Line
 	6400 2450 7200 2450
-Connection ~ 7200 2400
-Connection ~ 7600 2100
 Wire Wire Line
 	8000 1800 8000 2650
 Wire Wire Line
 	6400 2650 8000 2650
-Connection ~ 8000 1800
 Wire Wire Line
 	8400 1500 8400 2750
 Wire Wire Line
 	6400 2750 8400 2750
-Connection ~ 8400 1500
 Wire Wire Line
 	6800 1100 6800 1300
 Wire Wire Line
 	6800 2200 6900 2200
-Connection ~ 6900 2200
 Wire Wire Line
 	7300 1900 6800 1900
-Connection ~ 7300 1900
 Connection ~ 6800 1900
 Wire Wire Line
@@
 Wire Wire Line
 	7700 1600 6800 1600
-Connection ~ 7700 1600
 Connection ~ 6800 1600
 Wire Wire Line
@@
 Wire Wire Line
 	8100 1300 6800 1300
-Connection ~ 8100 1300
 Connection ~ 6800 1300
 Wire Wire Line
@@
 Wire Wire Line
 	8800 2200 8800 2250
-Connection ~ 7500 2200
 Wire Wire Line
 	7900 1900 8800 1900
 Wire Wire Line
 	8800 1900 8800 2200
-Connection ~ 7900 1900
 Connection ~ 8800 2200
 Wire Wire Line
@@
 Wire Wire Line
 	8800 1600 8800 1900
-Connection ~ 8300 1600
 Connection ~ 8800 1900
 Wire Wire Line
@@
 Wire Wire Line
 	8800 1300 8800 1600
-Connection ~ 8700 1300
 Connection ~ 8800 1600
 Wire Wire Line
@@
 	3700 3900 3700 4000
 $Comp
-L power:GND #PWR027
+L power:GND #PWR032
 U 1 1 5E39962F
 P 3700 4000
-F 0 "#PWR027" H 3700 3750 50  0001 C CNN
+F 0 "#PWR032" H 3700 3750 50  0001 C CNN
 F 1 "GND" H 3700 3850 50  0000 C CNN
 F 2 "" H 3700 4000 50  0001 C CNN
@@
 $EndComp
 $Comp
-L power:+3V3 #PWR026
+L power:+3V3 #PWR031
 U 1 1 5E3A0F34
 P 3700 3600
-F 0 "#PWR026" H 3700 3450 50  0001 C CNN
+F 0 "#PWR031" H 3700 3450 50  0001 C CNN
 F 1 "+3V3" H 3700 3740 50  0000 C CNN
 F 2 "" H 3700 3600 50  0001 C CNN
@@
 $EndComp
 $Comp
-L power:GND #PWR025
+L power:GND #PWR030
 U 1 1 5E3B7BFA
 P 2750 4400
-F 0 "#PWR025" H 2750 4150 50  0001 C CNN
+F 0 "#PWR030" H 2750 4150 50  0001 C CNN
 F 1 "GND" H 2750 4250 50  0000 C CNN
 F 2 "" H 2750 4400 50  0001 C CNN
@@
 $EndComp
 $Comp
-L power:+3V3 #PWR024
+L power:+3V3 #PWR029
 U 1 1 5E3BE166
 P 2750 3000
-F 0 "#PWR024" H 2750 2850 50  0001 C CNN
+F 0 "#PWR029" H 2750 2850 50  0001 C CNN
 F 1 "+3V3" H 2750 3140 50  0000 C CNN
 F 2 "" H 2750 3000 50  0001 C CNN
@@
 	2750 3600 2750 3700
 $Comp
-L Device:R R7
+L Device:R R14
 U 1 1 5E40139B
 P 1950 4550
-F 0 "R7" H 2020 4596 50  0000 L CNN
+F 0 "R14" H 2020 4596 50  0000 L CNN
 F 1 "10k" H 2020 4505 50  0000 L CNN
 F 2 "Resistor_SMD:R_1206_3216Metric_Pad1.42x1.75mm_HandSolder" V 1880 4550 50  0001 C CNN
@@
 $EndComp
 $Comp
-L Device:R R6
+L Device:R R13
 U 1 1 5E40263A
 P 1650 4550
-F 0 "R6" H 1720 4596 50  0000 L CNN
+F 0 "R13" H 1720 4596 50  0000 L CNN
 F 1 "10k" H 1720 4505 50  0000 L CNN
 F 2 "Resistor_SMD:R_1206_3216Metric_Pad1.42x1.75mm_HandSolder" V 1580 4550 50  0001 C CNN
@@
 $EndComp
 $Comp
-L Device:R R5
+L Device:R R12
 U 1 1 5E4081A2
 P 1350 4550
-F 0 "R5" H 1420 4596 50  0000 L CNN
+F 0 "R12" H 1420 4596 50  0000 L CNN
 F 1 "10k" H 1420 4505 50  0000 L CNN
 F 2 "Resistor_SMD:R_1206_3216Metric_Pad1.42x1.75mm_HandSolder" V 1280 4550 50  0001 C CNN
@@
 $EndComp
 $Comp
-L power:GND #PWR023
+L power:GND #PWR028
 U 1 1 5E40ED05
 P 1950 4900
-F 0 "#PWR023" H 1950 4650 50  0001 C CNN
+F 0 "#PWR028" H 1950 4650 50  0001 C CNN
 F 1 "GND" H 1950 4750 50  0000 C CNN
 F 2 "" H 1950 4900 50  0001 C CNN
@@
 Text HLabel 9000 2750 2    60   BiDi ~ 0
 ADC4
+$Comp
+L Diode:BAT54S D3
+U 1 1 5E211E6E
+P 8000 1600
+F 0 "D3" V 7954 1688 50  0000 L CNN
+F 1 "BAT54S" V 8045 1688 50  0000 L CNN
+F 2 "Package_TO_SOT_SMD:SOT-23" H 8075 1725 50  0001 L CNN
+F 3 "https://www.diodes.com/assets/Datasheets/ds11005.pdf" H 7880 1600 50  0001 C CNN
+	1    8000 1600
+	-1   0    0    -1
+$EndComp
+$Comp
+L Diode:BAT54S D4
+U 1 1 5E211E70
+P 8400 1300
+F 0 "D4" V 8354 1388 50  0000 L CNN
+F 1 "BAT54S" V 8445 1388 50  0000 L CNN
+F 2 "Package_TO_SOT_SMD:SOT-23" H 8475 1425 50  0001 L CNN
+F 3 "https://www.diodes.com/assets/Datasheets/ds11005.pdf" H 8280 1300 50  0001 C CNN
+	1    8400 1300
+	-1   0    0    -1
+$EndComp
 $EndSCHEMATC
