File: Flight Computer.kicad_pcb (KiCad board)
At the start: 4 copper layers, 27.5 x 83.3 mm, 92 parts, among them J1 Conn_01x08, J2 JTAG, J3 PAYLOAD, Q1 DMP3099, Q2 2N7002, Q3 2N7002, Q4 2N7002, Q5 DMP3099, Q6 DMP3099, SW1 Reset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

Commit message: Add pin labels to silkscreen
Parts:
- moved G1 0.51 mm to (68.1, 52.6)
Other:
- board text added: "AUX"
- board text added: "BATT"
- board text added: "DEPLOY"
- board text added: "DROGUE"
- board text added: "GND"
- board text added: "MAIN"
- board text added: "SCL"
- board text added: "SDA"
Changed lines of the file:
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@@
-(kicad_pcb (version 20171130) (host pcbnew "(5.1.5)-3")
+(kicad_pcb (version 20171130) (host pcbnew 5.1.5)
   (general
     (thickness 1.6)
-    (drawings 9)
+    (drawings 21)
     (tracks 940)
     (zones 0)
@@
   )
   (module Flight-Computer:SEDS_logo_soldermask (layer B.Cu)
-    (at 68.072 52.07 180)
+    (at 68.072 52.578 180)
     (fp_text reference G1 (at 0 0 180) (layer B.SilkS) hide
       (effects (font (size 0.762 0.762) (thickness 0.1524)) (justify mirror))
@@
     (pad 1 np_thru_hole circle (at 0 0) (size 2.5 2.5) (drill 2.5) (layers *.Cu *.Mask))
   )
-  (gr_text "Flight Computer Rev 4" (at 66.04 54.102) (layer B.Mask)
+  (gr_text DEPLOY (at 60.452 53.34) (layer B.SilkS)
+    (effects (font (size 0.508 0.508) (thickness 0.127)) (justify right mirror))
+  )
+  (gr_text SCL (at 60.452 52.07) (layer B.SilkS)
+    (effects (font (size 0.508 0.508) (thickness 0.127)) (justify right mirror))
+  )
+  (gr_text SDA (at 57.658 52.07) (layer B.SilkS)
+    (effects (font (size 0.508 0.508) (thickness 0.127)) (justify left mirror))
+  )
+  (gr_text GND (at 57.658 53.594) (layer B.SilkS)
+    (effects (font (size 0.508 0.508) (thickness 0.127)) (justify left mirror))
+  )
+  (gr_text AUX (at 59.944 129.54 270) (layer B.SilkS)
+    (effects (font (size 0.762 0.762) (thickness 0.1524)) (justify left mirror))
+  )
+  (gr_text MAIN (at 65.024 129.54 270) (layer B.SilkS)
+    (effects (font (size 0.762 0.762) (thickness 0.1524)) (justify left mirror))
+  )
+  (gr_text DROGUE (at 70.104 129.54 270) (layer B.SilkS)
+    (effects (font (size 0.762 0.762) (thickness 0.1524)) (justify left mirror))
+  )
+  (gr_text BATT (at 75.184 129.54 270) (layer B.SilkS)
+    (effects (font (size 0.762 0.762) (thickness 0.1524)) (justify left mirror))
+  )
+  (gr_text GND (at 72.644 129.54 270) (layer B.SilkS)
+    (effects (font (size 0.762 0.762) (thickness 0.1524)) (justify left mirror))
+  )
+  (gr_text GND (at 67.564 129.54 270) (layer B.SilkS)
+    (effects (font (size 0.762 0.762) (thickness 0.1524)) (justify left mirror))
+  )
+  (gr_text GND (at 62.484 129.54 270) (layer B.SilkS)
+    (effects (font (size 0.762 0.762) (thickness 0.1524)) (justify left mirror))
+  )
+  (gr_text GND (at 57.404 129.54 270) (layer B.SilkS)
+    (effects (font (size 0.762 0.762) (thickness 0.1524)) (justify left mirror))
+  )
+  (gr_text "Flight Computer Rev 4" (at 66.04 56.642) (layer B.Mask)
     (effects (font (size 0.635 0.635) (thickness 0.127)) (justify mirror))
   )
